File: meepolab pcb/meepolab pcb.kicad_pcb (KiCad board)
At the start: 4 copper layers, 193 parts, among them J1 Conn_01x12_Socket, J10 Conn_01x12_Socket, J11 Conn_01x12_Socket, J12 Conn_01x12_Socket, J13 Piezo socket, J14 Piezo socket, J15 Piezo socket, J16 Piezo socket, J17 Piezo socket, J18 Piezo socket, J19 Piezo socket, J2 Conn_01x12_Socket, J20 Piezo socket, J21 Conn_01x12_Socket, J3 Conn_01x12_Socket, J4 Conn_01x12_Socket, J5 Conn_01x12_Socket, J6 Conn_01x12_Socket, J7 Conn_01x12_Socket, J8 Conn_01x12_Socket, J9 Conn_01x12_Socket, U1 Teensy4.1, U2 CD74HC4067M, U3 CD74HC4067M, U4 74HC595, U5 74HC595, U6 74HC595, U7 74HC595

Commit message: wokred on routing
Parts:
- added H3: MountingHole_Pad, TestPoint:TestPoint_Pad_1.0x1.0mm, F.Cu at (203.0, 99.5)
- added H4: MountingHole_Pad, TestPoint:TestPoint_Pad_1.0x1.0mm, F.Cu at (200.5, 99.5)
- C1, C10, C2, C3, C5, C6, D104, D105, D106, D83, D84, D85, D89, D90, D91, D92, D93, D94, H1, H2, R1, R2, R35, R37, R38, R42: moved to B.Cu
- moved D74 72.4 mm to (247.6, 97.0)
- moved D73 71.0 mm to (242.6, 97.0)
- moved D68 61.8 mm to (247.6, 92.0)
- moved D67 60.1 mm to (242.6, 92.0)
- moved D66 59.0 mm to (237.6, 92.0)
- moved D65 58.4 mm to (232.6, 92.0)
- moved D81 53.7 mm to (189.1, 97.0)
- moved D41 52.6 mm to (242.5, 87.0)
- moved D82 50.8 mm to (194.1, 97.0)
- moved J15 50.6 mm to (221.2, 45.5), turned to 0 degrees
- moved D72 49.8 mm to (237.6, 97.0)
- moved D107 48.3 mm to (199.1, 97.0)
- moved D71 48.3 mm to (232.6, 97.0)
- moved D70 47.5 mm to (227.6, 97.0)
- moved D69 47.4 mm to (222.6, 97.0)
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Connections:
- J12 pad 10: unconnected-(J12-Pin_10-Pad10) -> Col10
- J12 pad 11: unconnected-(J12-Pin_11-Pad11) -> RecGnd
- J12 pad 12: unconnected-(J12-Pin_12-Pad12) -> Col10
- J12 pad 5: unconnected-(J12-Pin_5-Pad5) -> ShiftGnd
- J12 pad 6: unconnected-(J12-Pin_6-Pad6) -> Col10
- J12 pad 7: unconnected-(J12-Pin_7-Pad7) -> OctUpGnd
- J12 pad 8: unconnected-(J12-Pin_8-Pad8) -> Col10
- J12 pad 9: unconnected-(J12-Pin_9-Pad9) -> OctDwnGnd
- U1 pad 20: unconnected-(U1-28_RX7-Pad20) -> Col6
- U1 pad 21: unconnected-(U1-29_TX7-Pad21) -> Col7
- U1 pad 22: unconnected-(U1-30_CRX3-Pad22) -> Col8
- U1 pad 26: unconnected-(U1-34_RX8-Pad26) -> Col10
- U1 pad 27: unconnected-(U1-35_TX8-Pad27) -> Col9
- U1 pad 29: Col10 -> Col5
Routing:
- net Row0: track 0.00 -> 214.1 mm, vias 0 -> 12
- net Row2: track 0.00 -> 208.9 mm, vias 0 -> 13
- net Row4: track 0.00 -> 206.3 mm, vias 0 -> 9
- net Row1: track 0.00 -> 196.8 mm, vias 0 -> 4
- net Row3: track 0.00 -> 196.8 mm, vias 0 -> 3
- net +3V3: track 80.6 -> 244.0 mm, vias 2 -> 12
- net Col1: track 0.00 -> 152.1 mm
- net Col2: track 0.00 -> 149.4 mm
- net Col0: track 0.00 -> 145.3 mm, vias 0 -> 2
- net Col7: track 0.00 -> 130.2 mm
- net Col8: track 0.00 -> 127.3 mm
- net S3_3: track 0.00 -> 127.1 mm, vias 0 -> 1
- net Col3: track 0.00 -> 124.1 mm
- net Col6: track 0.00 -> 122.1 mm, vias 0 -> 1
- net S3_1: track 0.00 -> 116.6 mm, vias 0 -> 2
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- added copper zone on B.Cu, net GND
- added copper zone on F.Cu, net GND
- added copper zone on In2.Cu, net GND
Other:
- board text added: "{ "ViaStitching": "0.2", "stitch_zone_0": { "HSpacing": "1", "VSpacing": "1", "HOffset": "0", "VOffset": "0", "Clearance": "0", "Randomize": false } }"
- board text added: "{ "ViaStitching": "0.2", "stitch_zone_0": { "HSpacing": "1", "VSpacing": "1", "HOffset": "1", "VOffset": "1", "Clearance": "0", "Randomize": false } }"
- board text added: "{ "ViaStitching": "0.2", "stitch_zone_0": { "HSpacing": "1.27", "VSpacing": "1.27", "HOffset": "0", "VOffset": "0", "Clearance": "0.2", "Randomize": false } }"
