File: meepolab pcb/meepolab pcb.kicad_sch (KiCad schematic)
At the start: 193 parts, among them J1 Conn_01x12_Socket, J10 Conn_01x12_Socket, J11 Conn_01x12_Socket, J12 Conn_01x12_Socket, J13 Piezo socket, J14 Piezo socket, J15 Piezo socket, J16 Piezo socket, J17 Piezo socket, J18 Piezo socket, J19 Piezo socket, J2 Conn_01x12_Socket, J20 Piezo socket, J21 Conn_01x12_Socket, J3 Conn_01x12_Socket, J4 Conn_01x12_Socket, J5 Conn_01x12_Socket, J6 Conn_01x12_Socket, J7 Conn_01x12_Socket, J8 Conn_01x12_Socket, J9 Conn_01x12_Socket, U1 Teensy4.1, U2 CD74HC4067M, U3 CD74HC4067M, U4 74HC595, U5 74HC595, U6 74HC595, U7 74HC595

Commit message: wokred on routing
Parts:
- added H3, H4: MountingHole_Pad, TestPoint:TestPoint_Pad_1.0x1.0mm, symbol Mechanical:MountingHole_Pad
Connections:
- net Col10: now also J12.10 (Pin_10), J12.12 (Pin_12), J12.6 (Pin_6), J12.8 (Pin_8), U1.26 (34_RX8), H4.1; no longer U1.29 (37_CS)
- net Col5: now also U1.29 (37_CS)
- net Col6: now also U1.20 (28_RX7)
- net Col7: now also U1.21 (29_TX7)
- net Col8: now also U1.22 (30_CRX3)
- net Col9: now also U1.27 (35_TX8)
- net OctDwnGnd: now also J12.9 (Pin_9)
- net OctUpGnd: now also J12.7 (Pin_7)
- net PlayPauseGnd: now also H3.1
- net RecGnd: now also J12.11 (Pin_11)
- net ShiftGnd: now also J12.5 (Pin_5)

Commit message: worked on layout
Parts:
- added J22: Conn_01x02_Socket, Connector_JST:JST_EH_B2B-EH-A_1x02_P2.50mm_Vertical, symbol Connector:Conn_01x02_Socket
Connections:
- net +3V3: no longer U4.16 (VCC), U5.16 (VCC), U6.16 (VCC), U7.16 (VCC)
- net GND: now also J22.2 (Pin_2)
- new net External 3v3: J22.1 (Pin_1), U4.16 (VCC), U5.16 (VCC), U6.16 (VCC), U7.16 (VCC)
